Commit message: create skills

File: sharework_cembre_description/urdf/sharework_cembre.xacro (robot description, xacro)
@@ -2,6 +2,6 @@
 <robot xmlns:xacro="http://ros.org/wiki/xacro" name="sharework" >
 <xacro:include filename="$(find ur_description)/urdf/ur5.urdf.xacro" />
-<xacro:include filename="$(find robotiq_85_description)/urdf/robotiq_85_gripper.urdf.xacro" />
 <xacro:include filename="$(find realsense2_description)/urdf/_d435.urdf.xacro" />
+<xacro:include filename="$(find robotiq_2f_85_gripper_visualization)/urdf/robotiq_arg2f_85_model_macro.xacro" />
 <xacro:property name="column_size_x" value="0.580" />
 <xacro:property name="column_size_y" value="0.120" />
@@ -23,5 +23,6 @@
 <xacro:property name="guide_size_y" value="${beam_size_y}" />
 <xacro:property name="guide_size_z" value="0.14" />
-<xacro:property name="guide_distance_x" value="0.105" />
+<xacro:property name="guide_distance_x" value="0.185" />
+<xacro:property name="anti_crushing_distance" value="0.020" />
 <xacro:property name="guide_distance_y" value="${0.385+0.041}" />
 <xacro:property name="wall_size_x" value="0.1" />
@@ -32,4 +33,6 @@
 <xacro:property name="floor_size_y" value="6" />
 <xacro:property name="floor_size_z" value="0.01" />
+<xacro:property name="virtual_wall_width" value="0.001" />
+<xacro:property name="virtual_wall2_gap" value="0.10" />
 <!-- electric plug cabinet -->
 <xacro:property name="ec_size_x" value="0.40" />
@@ -39,4 +42,5 @@
 <xacro:property name="beech" value="0.952941176470588	0.694117647058823	0.392156862745098 1" />
 <xacro:property name="floor" value="0.4 0.4 0.5 1" />
+<xacro:property name="virtual_wall" value="1 0.2 0.2 0.2" />
 <link name="world"/>
   <joint name="base_to_right_leg" type="fixed">
@@ -70,4 +74,15 @@
      <origin xyz="${0.5*column_size_x} ${0.5*column_size_y} ${0.5*column_size_z}" rpy="0 0 0" />
      <geometry>
+       <box size="${column_size_x+2*anti_crushing_distance} ${column_size_y+2*anti_crushing_distance} ${column_size_z}" />
+     </geometry>
+     <material name="Grey">
+       <color rgba="${grey}"/>
+     </material>
+   </collision>
+</link>
+<link name="left_column">
+   <visual>
+     <origin xyz="${0.5*column_size_x} ${-0.5*column_size_y} ${0.5*column_size_z}" rpy="0 0 0" />
+     <geometry>
        <box size="${column_size_x} ${column_size_y} ${column_size_z}" />
      </geometry>
@@ -75,20 +90,9 @@
        <color rgba="${grey}"/>
      </material>
-   </collision>
-</link>
-<link name="left_column">
-   <visual>
+   </visual>
+   <collision>
      <origin xyz="${0.5*column_size_x} ${-0.5*column_size_y} ${0.5*column_size_z}" rpy="0 0 0" />
      <geometry>
-       <box size="${column_size_x} ${column_size_y} ${column_size_z}" />
-     </geometry>
-     <material name="Grey">
-       <color rgba="${grey}"/>
-     </material>
-   </visual>
-   <collision>
-     <origin xyz="${0.5*column_size_x} ${-0.5*column_size_y} ${0.5*column_size_z}" rpy="0 0 0" />
-     <geometry>
-       <box size="${column_size_x} ${column_size_y} ${column_size_z}" />
+       <box size="${column_size_x+2*anti_crushing_distance} ${column_size_y+2*anti_crushing_distance} ${column_size_z}" />
      </geometry>
      <material name="Grey">
@@ -106,5 +110,5 @@
      <origin xyz="${0.5*beam_size_x} 0 ${-0.5*beam_size_z}" rpy="0 0 0" />
      <geometry>
-       <box size="${beam_size_x} ${beam_size_y} ${beam_size_z}" />
+       <box size="${beam_size_x} ${beam_size_y} ${beam_size_z+2*anti_crushing_distance}" />
      </geometry>
      <material name="Grey">
@@ -219,5 +223,5 @@
      <origin xyz="${0.5*table_size_x} ${0.5*table_size_y} ${-0.5*table_size_z}" rpy="0 0 0" />
      <geometry>
-       <box size="${table_size_x} ${table_size_y} ${table_size_z}" />
+       <box size="${table_size_x} ${table_size_y} ${table_size_z+anti_crushing_distance}" />
      </geometry>
      <material name="Beech">
@@ -353,5 +357,4 @@
     <origin xyz="0.0 0.0 0.0" rpy="0 0 ${0.0*pi}" />
   </joint>
-  <xacro:include filename="$(find robotiq_2f_85_gripper_visualization)/urdf/robotiq_arg2f_85_model_macro.xacro" />
   <xacro:robotiq_arg2f_85 prefix=""/>
 <link name="open_tip" />
@@ -367,4 +370,29 @@
   <origin xyz="0 0 0.163" rpy="0 0 ${0.5*pi}" />
 </joint>
+<joint name="rq_connector_joint" type="fixed">
+<parent link="robotiq_coupler" />
+<child  link = "rq_connector" />
+<origin xyz="-0.06 0 0" rpy="0 0 0" />
+</joint>
+<link name="rq_connector">
+   <visual>
+     <origin xyz="0 0 0" rpy="0 0 0" />
+     <geometry>
+       <box size="0.04 0.04 0.04" />
+     </geometry>
+     <material name="White">
+       <color rgba="1 1 1 1"/>
+     </material>
+   </visual>
+   <collision>
+   <origin xyz="0 0 0" rpy="0 0 0" />
+   <geometry>
+     <box size="0.04 0.04 0.04" />
+   </geometry>
+   <material name="White">
+     <color rgba="1 1 1 1"/>
+   </material>
+   </collision>
+</link>
 <!-- walls  -->
 <joint name="portal_to_wall" type="fixed">
@@ -418,5 +446,5 @@
    </collision>
 </link>
-<joint name="portal_to_flor" type="fixed">
+<joint name="portal_to_floor" type="fixed">
     <parent link="portal"/>
     <child link="floor"/>
@@ -442,4 +470,55 @@
    </material>
    </collision>
+</link>
+<!-- Virtual Wall -->
+<joint name="virtual_wall_1_joint" type="fixed">
+    <parent link="guide_fixed"/>
+    <child link="virtual_wall_1"/>
+    <origin xyz="0 0 0.20"/>
+  </joint>
+<link name="virtual_wall_1">
+   <visual>
+     <origin xyz="0 ${0.5*beam_size_y} ${+0.5*virtual_wall_width}" rpy="0 0 0" />
+     <geometry>
+       <box size="${0.2+column_size_x} ${beam_size_y+2*column_size_y} ${virtual_wall_width}" />
+     </geometry>
+     <material name="VirtualWallColor">
+       <color rgba="${virtual_wall}"/>
+     </material>
+   </visual>
+<collision>
+<origin xyz="0 ${0.5*beam_size_y} ${+0.5*virtual_wall_width}" rpy="0 0 0" />
+<geometry>
+<box size="${0.2+column_size_x} ${beam_size_y+2*column_size_y} ${virtual_wall_width}" />
+</geometry>
+<material name="VirtualWallColor">
+  <color rgba="${virtual_wall}"/>
+</material>
+</collision>
+</link>
+<joint name="virtual_wall_2_joint" type="fixed">
+    <parent link="world"/>
+    <child link="virtual_wall_2"/>
+    <origin xyz="${table_size_x+virtual_wall2_gap} 0 0.0"/>
+  </joint>
+<link name="virtual_wall_2">
+   <visual>
+     <origin xyz="${0.5*virtual_wall_width} 0 1" rpy="0 0 0" />
+     <geometry>
+       <box size="${virtual_wall_width} ${beam_size_y+2*column_size_y} 2" />
+     </geometry>
+     <material name="VirtualWallColor">
+       <color rgba="${virtual_wall}"/>
+     </material>
+   </visual>
+<collision>
+<origin xyz="${0.5*virtual_wall_width} 0 1" rpy="0 0 0" />
+<geometry>
+  <box size="${virtual_wall_width} ${beam_size_y+2*column_size_y} 2" />
+</geometry>
+<material name="VirtualWallColor">
+  <color rgba="${virtual_wall}"/>
+</material>
+</collision>
 </link>
 <!-- CAMERA -->

Commit message: add skills

File: sharework_cembre_description/urdf/sharework_cembre.xacro (robot description, xacro)
@@ -351,4 +351,8 @@
      </material>
 </collision>
+<inertial>
+  <mass value="0.5"/>
+  <inertia ixx="0.1" ixy="0.0" ixz="0.0" iyy="0.1" iyz="0.0" izz="0.4"/>
+</inertial>
 </link>
     <joint name="robotiq_joint" type="fixed">
@@ -478,13 +482,4 @@
   </joint>
 <link name="virtual_wall_1">
-   <visual>
-     <origin xyz="0 ${0.5*beam_size_y} ${+0.5*virtual_wall_width}" rpy="0 0 0" />
-     <geometry>
-       <box size="${0.2+column_size_x} ${beam_size_y+2*column_size_y} ${virtual_wall_width}" />
-     </geometry>
-     <material name="VirtualWallColor">
-       <color rgba="${virtual_wall}"/>
-     </material>
-   </visual>
 <collision>
 <origin xyz="0 ${0.5*beam_size_y} ${+0.5*virtual_wall_width}" rpy="0 0 0" />
@@ -503,13 +498,4 @@
   </joint>
 <link name="virtual_wall_2">
-   <visual>
-     <origin xyz="${0.5*virtual_wall_width} 0 1" rpy="0 0 0" />
-     <geometry>
-       <box size="${virtual_wall_width} ${beam_size_y+2*column_size_y} 2" />
-     </geometry>
-     <material name="VirtualWallColor">
-       <color rgba="${virtual_wall}"/>
-     </material>
-   </visual>
 <collision>
 <origin xyz="${0.5*virtual_wall_width} 0 1" rpy="0 0 0" />

Commit message: change rs camera position

File: sharework_cembre_description/urdf/sharework_cembre.xacro (robot description, xacro)
@@ -466,7 +466,33 @@
    </visual>
    <collision>
-   <origin xyz="${0.5*floor_size_x-column_size_x-wall_distance} 0 0.2" rpy="0 0 0" />
-   <geometry>
-     <box size="${floor_size_x} ${floor_size_y} ${.4}" />
+   <origin xyz="${0.5*floor_size_x-column_size_x-wall_distance} 0 0.4" rpy="0 0 0" />
+   <geometry>
+     <box size="${floor_size_x} ${floor_size_y} ${.8}" />
+   </geometry>
+   <material name="White">
+     <color rgba="1 1 1 1"/>
+   </material>
+   </collision>
+</link>
+<!-- Screw driver -->
+<joint name="table_to_screwdriver_holder" type="fixed">
+    <parent link="table"/>
+    <child link="screwdriver_holder"/>
+    <origin xyz="0.2 -0.05 1.5"/>
+  </joint>
+<link name="screwdriver_holder">
+   <visual>
+     <origin xyz="0 0 0" rpy="0 0 0" />
+     <geometry>
+       <box size="0.4 0.2 1.5" />
+     </geometry>
+     <material name="White">
+       <color rgba="1 1 1 1"/>
+     </material>
+   </visual>
+   <collision>
+   <origin xyz="0 0 0" rpy="0 0 0" />
+   <geometry>
+     <box size="0.2 0.2 2" />
    </geometry>
    <material name="White">
@@ -510,11 +536,11 @@
 <!-- CAMERA -->
 <joint name="upper_beam_to_realsense2" type="fixed">
-    <parent link="upper_beam"/>
+    <parent link="table"/>
     <child link="realsense_holder1"/>
-    <origin xyz="0.62 0 0" rpy="0 ${pi/3.0} 0"/>
+    <origin xyz="0.578 2.040 1.742" rpy="0.008 0.662 -1.725"/>
   </joint>
 <link name="realsense_holder1"/>
- <sensor_d435 parent="realsense_holder1">
+ <xacro:sensor_d435 parent="realsense_holder1" use_nominal_extrinsics="false">
    <origin xyz="0 0 0" rpy="0 0 0"/>
- </sensor_d435>
+ </xacro:sensor_d435>
 </robot>

Commit message: add pickplace test

File: sharework_cembre_description/urdf/sharework_cembre.xacro (robot description, xacro)
@@ -1,5 +1,4 @@
 <?xml version="1.0"?>
 <robot xmlns:xacro="http://ros.org/wiki/xacro" name="sharework" >
-<xacro:include filename="$(find ur_description)/urdf/ur5.urdf.xacro" />
 <xacro:include filename="$(find realsense2_description)/urdf/_d435.urdf.xacro" />
 <xacro:include filename="$(find robotiq_2f_85_gripper_visualization)/urdf/robotiq_arg2f_85_model_macro.xacro" />
@@ -16,5 +15,5 @@
 <xacro:property name="rail_size_x" value="0.36" />
 <xacro:property name="rail_size_y" value="3.224" />
-<xacro:property name="rail_size_z" value="0.11" />
+<xacro:property name="rail_size_z" value="0.17" />
 <xacro:property name="rail_distance" value="${0.162+0.5*rail_size_x}" />
 <xacro:property name="upper_beam_height" value="2.208" />
@@ -223,5 +222,5 @@
      <origin xyz="${0.5*table_size_x} ${0.5*table_size_y} ${-0.5*table_size_z}" rpy="0 0 0" />
      <geometry>
-       <box size="${table_size_x} ${table_size_y} ${table_size_z+anti_crushing_distance}" />
+       <box size="${table_size_x} ${table_size_y} ${table_size_z}" />
      </geometry>
      <material name="Beech">
@@ -264,6 +263,6 @@
     shoulder_lift_lower_limit="${-2*pi}" shoulder_lift_upper_limit="${2*pi}"
     elbow_joint_lower_limit="${-pi}" elbow_joint_upper_limit="${2*pi}"
-    wrist_1_lower_limit="${-2*pi}" wrist_1_upper_limit="${2*pi}"
-    wrist_2_lower_limit="${-2*pi}" wrist_2_upper_limit="${2*pi}"
+    wrist_1_lower_limit="${-pi}" wrist_1_upper_limit="${pi}"
+    wrist_2_lower_limit="${-pi}" wrist_2_upper_limit="${pi}"
     wrist_3_lower_limit="${-2*pi}" wrist_3_upper_limit="${2*pi}"
     transmission_hw_interface="$(arg transmission_hw_interface)"

Commit message: update configurations

File: sharework_cembre_description/urdf/sharework_cembre.xacro (robot description, xacro)
@@ -28,10 +28,10 @@
 <xacro:property name="wall_size_y" value="${2+table_size_y+2*column_size_y}" />
 <xacro:property name="wall_size_z" value="${column_size_z}" />
-<xacro:property name="wall_distance" value="0.680" />
+<xacro:property name="wall_distance" value="0.500" />
 <xacro:property name="floor_size_x" value="6" />
 <xacro:property name="floor_size_y" value="6" />
 <xacro:property name="floor_size_z" value="0.01" />
 <xacro:property name="virtual_wall_width" value="0.001" />
-<xacro:property name="virtual_wall2_gap" value="0.10" />
+<xacro:property name="virtual_wall2_gap" value="1.10" />
 <!-- electric plug cabinet -->
 <xacro:property name="ec_size_x" value="0.40" />
@@ -169,5 +169,5 @@
    <origin xyz="0 ${0.5*guide_size_y} ${+0.5*guide_size_z}" rpy="0 0 0" />
    <geometry>
-     <box size="${guide_size_x} ${guide_size_y} ${guide_size_z}" />
+     <box size="${guide_size_x+0.3} ${guide_size_y} ${guide_size_z}" />
    </geometry>
    <material name="Grey">
@@ -262,7 +262,7 @@
     shoulder_pan_lower_limit="${-2*pi}" shoulder_pan_upper_limit="${2*pi}"
     shoulder_lift_lower_limit="${-2*pi}" shoulder_lift_upper_limit="${2*pi}"
-    elbow_joint_lower_limit="${-pi}" elbow_joint_upper_limit="${2*pi}"
-    wrist_1_lower_limit="${-pi}" wrist_1_upper_limit="${pi}"
-    wrist_2_lower_limit="${-pi}" wrist_2_upper_limit="${pi}"
+    elbow_joint_lower_limit="${-2*pi}" elbow_joint_upper_limit="${2*pi}"
+    wrist_1_lower_limit="${-2*pi}" wrist_1_upper_limit="${2*pi}"
+    wrist_2_lower_limit="${-2*pi}" wrist_2_upper_limit="${2*pi}"
     wrist_3_lower_limit="${-2*pi}" wrist_3_upper_limit="${2*pi}"
     transmission_hw_interface="$(arg transmission_hw_interface)"
@@ -504,11 +504,11 @@
     <parent link="guide_fixed"/>
     <child link="virtual_wall_1"/>
-    <origin xyz="0 0 0.20"/>
+    <origin xyz="0 0 0.0"/>
   </joint>
 <link name="virtual_wall_1">
 <collision>
-<origin xyz="0 ${0.5*beam_size_y} ${+0.5*virtual_wall_width}" rpy="0 0 0" />
+<origin xyz="-0.4 ${0.5*beam_size_y} ${+0.5*virtual_wall_width}" rpy="0 0 0" />
 <geometry>
-<box size="${0.2+column_size_x} ${beam_size_y+2*column_size_y} ${virtual_wall_width}" />
+<box size="${1.0+column_size_x} ${beam_size_y+2*column_size_y} ${virtual_wall_width}" />
 </geometry>
 <material name="VirtualWallColor">

Commit message: modified config files

File: sharework_cembre_description/urdf/sharework_cembre.xacro (robot description, xacro)
@@ -291,5 +291,5 @@
 </visual>
 <collision>
-<origin xyz="0 0 0.005" rpy="0 0 0" />
+<origin xyz="0 0 0.005" rpy="0 ${0.5*pi} 0" />
  <geometry>
   <cylinder radius="${0.10*0.5}" length="0.30"/>
