Commit message: add simplified collisions

File: sharework_cembre_description/urdf/sharework_cembre_simplified.xacro (robot description, xacro)
@@ -1,4 +1,4 @@
 <?xml version="1.0"?>
-<robot xmlns:xacro="http://ros.org/wiki/xacro" name="sharework" >
+<robot xmlns:xacro="http://ros.org/wiki/xacro" name="sharework_simplified" >
 <xacro:include filename="$(find realsense2_description)/urdf/_d435.urdf.xacro" />
 <xacro:include filename="$(find robotiq_2f_85_gripper_visualization)/urdf/robotiq_arg2f_85_model_macro.xacro" />
@@ -41,5 +41,4 @@
 <xacro:property name="beech" value="0.952941176470588	0.694117647058823	0.392156862745098 1" />
 <xacro:property name="floor" value="0.4 0.4 0.5 1" />
-<xacro:property name="virtual_wall" value="1 0.2 0.2 0.2" />
 <link name="world"/>
   <joint name="base_to_right_leg" type="fixed">
@@ -204,9 +203,9 @@
 </link>
 <!-- TABLE -->
-  <joint name="portal_to_table" type="fixed">
-    <parent link="world"/>
-    <child link="table"/>
-    <origin xyz="0 ${-0.5*table_size_y} ${table_height}"/>
-  </joint>
+<joint name="portal_to_table" type="fixed">
+  <parent link="world"/>
+  <child link="table"/>
+  <origin xyz="0 ${-0.5*table_size_y} ${table_height}"/>
+</joint>
 <link name="table">
    <visual>
@@ -254,148 +253,24 @@
    </collision>
 </link>
-  <!-- ur10e -->
-  <xacro:include filename="$(find ur_e_description)/urdf/ur10e.urdf.xacro" />
-  <xacro:arg name="transmission_hw_interface" default="hardware_interface/PositionJointInterface"/>
-  <!-- arm -->
-  <xacro:arg name="kinematics_config" default="$(find sharework_cembre_description)/config/cembre_ur10e.yaml"/>
-  <xacro:ur10e_robot prefix="" joint_limited="true"
-    shoulder_pan_lower_limit="${-2*pi}" shoulder_pan_upper_limit="${2*pi}"
-    shoulder_lift_lower_limit="${-2*pi}" shoulder_lift_upper_limit="${2*pi}"
-    elbow_joint_lower_limit="${-2*pi}" elbow_joint_upper_limit="${2*pi}"
-    wrist_1_lower_limit="${-2*pi}" wrist_1_upper_limit="${2*pi}"
-    wrist_2_lower_limit="${-2*pi}" wrist_2_upper_limit="${2*pi}"
-    wrist_3_lower_limit="${-2*pi}" wrist_3_upper_limit="${2*pi}"
-    transmission_hw_interface="$(arg transmission_hw_interface)"
-    kinematics_file="${load_yaml('$(arg kinematics_config)')}"
-    />
-  <joint name="cursor_to_base" type="fixed">
-    <parent link="cursor" />
-    <child link = "base_link" />
-    <origin xyz="0.0 0.0 0.0" rpy="${pi} 0.0 ${0.5*pi}" />
-  </joint>
-<!-- gripper -->
-<joint name="anti_clamping_joint" type="fixed">
-<parent link="forearm_link" />
-<child  link = "anti_clamping_obstacle" />
-<origin xyz="-0.45 0 0.03" rpy="0 0 0" />
+<!-- ur10e -->
+<xacro:include filename="$(find ur10e_robotiq_simplified_description)/urdf/ur10e_robotiq.urdf.xacro" />
+<xacro:arg name="transmission_hw_interface" default="hardware_interface/PositionJointInterface"/>
+<!-- arm -->
+<xacro:arg name="kinematics_config" default="$(find sharework_cembre_description)/config/cembre_ur10e.yaml"/>
+<xacro:ur10e_robot prefix="" joint_limited="true"
+  shoulder_pan_lower_limit="${-pi}" shoulder_pan_upper_limit="${pi}"
+  shoulder_lift_lower_limit="${-pi}" shoulder_lift_upper_limit="0.05"
+  elbow_joint_lower_limit="${-pi}" elbow_joint_upper_limit="${pi}"
+  wrist_1_lower_limit="${-2*pi}" wrist_1_upper_limit="${2*pi}"
+  wrist_2_lower_limit="${-2*pi}" wrist_2_upper_limit="${2*pi}"
+  wrist_3_lower_limit="${-2*pi}" wrist_3_upper_limit="${2*pi}"
+  transmission_hw_interface="$(arg transmission_hw_interface)"
+  kinematics_file="${load_yaml('$(arg kinematics_config)')}"
+/>
+<joint name="cursor_to_base" type="fixed">
+  <parent link="cursor" />
+  <child link = "base_link" />
+  <origin xyz="0.0 0.0 0.0" rpy="${pi} 0.0 ${0.5*pi}" />
 </joint>
-<link name="anti_clamping_obstacle">
-<visual>
-  <origin xyz="0 0 0.000" rpy="0 ${0.5*pi} 0" />
-   <geometry>
-    <cylinder radius="${0.10*0.5}" length="0.30"/>
-   </geometry>
-   <material name="RobotiqGrey">
-     <color rgba="0.1 0.1 0.1 0.5"/>
-   </material>
-</visual>
-<collision>
-<origin xyz="0 0 0.005" rpy="0 ${0.5*pi} 0" />
- <geometry>
-  <cylinder radius="${0.10*0.5}" length="0.30"/>
- </geometry>
- <material name="RobotiqGrey">
-   <color rgba="0.1 0.1 0.1 0.5"/>
- </material>
-</collision>
-</link>
-<joint name="anti_clamping_joint2" type="fixed">
-<parent link="tool0" />
-<child  link = "anti_clamping_obstacle2" />
-<origin xyz="0 0 -0.06" rpy="0 0 0" />
-</joint>
-<link name="anti_clamping_obstacle2">
-<visual>
-  <origin xyz="0 0 0.000" rpy="0 0 0" />
-   <geometry>
-    <cylinder radius="${0.10*0.5}" length="0.12"/>
-   </geometry>
-   <material name="RobotiqGrey">
-     <color rgba="0.1 0.1 0.1 0.5"/>
-   </material>
-</visual>
-<collision>
-<origin xyz="0 0 0.005" rpy="0 0 0" />
- <geometry>
-  <cylinder radius="${0.10*0.5}" length="0.12"/>
- </geometry>
- <material name="RobotiqGrey">
-   <color rgba="0.1 0.1 0.1 0.5"/>
- </material>
-</collision>
-</link>
-  <!-- gripper -->
-<joint name="rq_coupler_joint" type="fixed">
-  <parent link="tool0" />
-  <child  link = "robotiq_coupler" />
-  <origin xyz="0 0 0.01" rpy="0 0 ${0.5*pi}" />
-</joint>
-<link name="robotiq_coupler">
-<visual>
-    <origin xyz="0 0 0.005" rpy="0 0 0" />
-     <geometry>
-      <cylinder radius="${0.075*0.5}" length="0.01"/>
-     </geometry>
-     <material name="RobotiqGrey">
-       <color rgba="0.1 0.1 0.1 1"/>
-     </material>
-</visual>
-<collision>
-    <origin xyz="0 0 0.005" rpy="0 0 0" />
-     <geometry>
-      <cylinder radius="${0.075*0.5}" length="0.01"/>
-     </geometry>
-     <material name="RobotiqGrey">
-       <color rgba="0.1 0.1 0.1 1"/>
-     </material>
-</collision>
-<inertial>
-  <mass value="0.5"/>
-  <inertia ixx="0.1" ixy="0.0" ixz="0.0" iyy="0.1" iyz="0.0" izz="0.4"/>
-</inertial>
-</link>
-    <joint name="robotiq_joint" type="fixed">
-    <parent link="robotiq_coupler" />
-    <child link = "robotiq_arg2f_base_link" />
-    <origin xyz="0.0 0.0 0.0" rpy="0 0 ${0.0*pi}" />
-  </joint>
-  <xacro:robotiq_arg2f_85 prefix=""/>
-<link name="open_tip" />
-<joint name="open_tip_joint" type="fixed">
-  <parent link="robotiq_coupler" />
-  <child  link = "open_tip" />
-  <origin xyz="0 0 0.149" rpy="0 0 ${0.5*pi}" />
-</joint>
-<link name="closed_tip" />
-<joint name="closed_tip_joint" type="fixed">
-  <parent link="robotiq_coupler" />
-  <child  link = "closed_tip" />
-  <origin xyz="0 0 0.163" rpy="0 0 ${0.5*pi}" />
-</joint>
-<joint name="rq_connector_joint" type="fixed">
-<parent link="robotiq_coupler" />
-<child  link = "rq_connector" />
-<origin xyz="-0.06 0 0" rpy="0 0 0" />
-</joint>
-<link name="rq_connector">
-   <visual>
-     <origin xyz="0 0 0" rpy="0 0 0" />
-     <geometry>
-       <box size="0.04 0.04 0.04" />
-     </geometry>
-     <material name="White">
-       <color rgba="1 1 1 1"/>
-     </material>
-   </visual>
-   <collision>
-   <origin xyz="0 0 0" rpy="0 0 0" />
-   <geometry>
-     <box size="0.04 0.04 0.04" />
-   </geometry>
-   <material name="White">
-     <color rgba="1 1 1 1"/>
-   </material>
-   </collision>
-</link>
 <!-- walls  -->
 <joint name="portal_to_wall" type="fixed">
@@ -428,5 +303,5 @@
     <child link="ec"/>
     <origin xyz="0 ${table_size_x*0.5} 0"/>
-  </joint>
+</joint>
 <link name="ec">
    <visual>
@@ -464,13 +339,4 @@
      </material>
    </visual>
-   <collision>
-   <origin xyz="${0.5*floor_size_x-column_size_x-wall_distance} 0 0.4" rpy="0 0 0" />
-   <geometry>
-     <box size="${floor_size_x} ${floor_size_y} ${.8}" />
-   </geometry>
-   <material name="White">
-     <color rgba="1 1 1 1"/>
-   </material>
-   </collision>
 </link>
 <!-- Screw driver -->
@@ -507,13 +373,13 @@
   </joint>
 <link name="virtual_wall_1">
-<collision>
-<origin xyz="-0.4 ${0.5*beam_size_y} ${+0.5*virtual_wall_width}" rpy="0 0 0" />
-<geometry>
-<box size="${1.0+column_size_x} ${beam_size_y+2*column_size_y} ${virtual_wall_width}" />
-</geometry>
-<material name="VirtualWallColor">
-  <color rgba="${virtual_wall}"/>
-</material>
-</collision>
+  <collision>
+    <origin xyz="-0.5 ${0.5*beam_size_y} ${+0.5*virtual_wall_width}" rpy="0 0 0" />
+    <geometry>
+      <box size="${1.0+column_size_x} ${beam_size_y+2*column_size_y} ${virtual_wall_width}" />
+    </geometry>
+    <material name="VirtualWallColor">
+      <color rgba="0.1 0.1 0.1 0.1"/>
+    </material>
+  </collision>
 </link>
 <joint name="virtual_wall_2_joint" type="fixed">
@@ -523,13 +389,13 @@
   </joint>
 <link name="virtual_wall_2">
-<collision>
-<origin xyz="${0.5*virtual_wall_width} 0 1" rpy="0 0 0" />
-<geometry>
-  <box size="${virtual_wall_width} ${beam_size_y+2*column_size_y} 2" />
-</geometry>
-<material name="VirtualWallColor">
-  <color rgba="${virtual_wall}"/>
-</material>
-</collision>
+  <collision>
+    <origin xyz="${0.5*virtual_wall_width} 0 1" rpy="0 0 0" />
+    <geometry>
+      <box size="${virtual_wall_width} ${beam_size_y+2*column_size_y} 2" />
+    </geometry>
+    <material name="VirtualWallColor2">
+      <color rgba="0.1 0.1 0.1 0.1"/>
+    </material>
+  </collision>
 </link>
 <!-- CAMERA -->
@@ -540,6 +406,6 @@
   </joint>
 <link name="realsense_holder1"/>
- <xacro:sensor_d435 parent="realsense_holder1" use_nominal_extrinsics="false">
-   <origin xyz="0 0 0" rpy="0 0 0"/>
- </xacro:sensor_d435>
+<xacro:sensor_d435 parent="realsense_holder1" use_nominal_extrinsics="false">
+  <origin xyz="0 0 0" rpy="0 0 0"/>
+</xacro:sensor_d435>
 </robot>

Commit message: guide moved

File: sharework_cembre_description/urdf/sharework_cembre_simplified.xacro (robot description, xacro)
@@ -18,4 +18,5 @@
 <xacro:property name="rail_distance" value="${0.162+0.5*rail_size_x}" />
 <xacro:property name="upper_beam_height" value="2.208" />
+<xacro:property name="guide_offset" value="0.70" />
 <xacro:property name="cursor_size" value="0.280" />
 <xacro:property name="guide_size_x" value="${cursor_size}" />
@@ -178,5 +179,5 @@
     <parent link="guide_fixed"/>
     <child link="cursor"/>
-    <origin xyz="0 ${guide_distance_y+0.5*cursor_size} -0.01"/>
+    <origin xyz="0 ${guide_distance_y+0.5*cursor_size} ${guide_offset}-0.01"/>
     <limit effort="1000.0" lower="0" upper="1.4" velocity="0.5"/>
     <axis xyz="0 1 0"/>

Commit message: moved cursor

File: sharework_cembre_description/urdf/sharework_cembre_simplified.xacro (robot description, xacro)
@@ -179,5 +179,5 @@
     <parent link="guide_fixed"/>
     <child link="cursor"/>
-    <origin xyz="0 ${guide_distance_y+0.5*cursor_size} ${guide_offset}-0.01"/>
+    <origin xyz="0 ${guide_distance_y+guide_offset+0.5*cursor_size} ${-0.01}"/>
     <limit effort="1000.0" lower="0" upper="1.4" velocity="0.5"/>
     <axis xyz="0 1 0"/>

Commit message: rviz

File: sharework_cembre_description/urdf/sharework_cembre_simplified.xacro (robot description, xacro)
@@ -18,5 +18,5 @@
 <xacro:property name="rail_distance" value="${0.162+0.5*rail_size_x}" />
 <xacro:property name="upper_beam_height" value="2.208" />
-<xacro:property name="guide_offset" value="0.70" />
+<xacro:property name="guide_offset" value="${0.70-0.205}" />
 <xacro:property name="cursor_size" value="0.280" />
 <xacro:property name="guide_size_x" value="${cursor_size}" />
@@ -261,5 +261,5 @@
 <xacro:ur10e_robot prefix="" joint_limited="true"
   shoulder_pan_lower_limit="${-pi}" shoulder_pan_upper_limit="${pi}"
-  shoulder_lift_lower_limit="${-pi}" shoulder_lift_upper_limit="0.05"
+  shoulder_lift_lower_limit="${-pi}" shoulder_lift_upper_limit="0.052359878"
   elbow_joint_lower_limit="${-pi}" elbow_joint_upper_limit="${pi}"
   wrist_1_lower_limit="${-pi}" wrist_1_upper_limit="${pi}"

Commit message: dual realsense

File: sharework_cembre_description/urdf/sharework_cembre_simplified.xacro (robot description, xacro)
@@ -24,5 +24,5 @@
 <xacro:property name="guide_size_z" value="0.14" />
 <xacro:property name="guide_distance_x" value="0.185" />
-<xacro:property name="anti_crushing_distance" value="0.020" />
+<xacro:property name="anti_crushing_distance" value="0.040" />
 <xacro:property name="guide_distance_y" value="${0.385+0.041}" />
 <xacro:property name="wall_size_x" value="0.1" />

Commit message: camera calib

File: sharework_cembre_description/urdf/sharework_cembre_simplified.xacro (robot description, xacro)
@@ -401,8 +401,8 @@
 </link>
 <!-- CAMERA -->
-<joint name="upper_beam_to_realsense2" type="fixed">
+<!--<joint name="upper_beam_to_realsense2" type="fixed">
     <parent link="table"/>
     <child link="realsense_holder1"/>
-    <origin xyz="0.578 2.040 1.742" rpy="0.008 0.662 -1.725"/>
+    <origin xyz="0.881438574717 0.787357038996 -0.685421164733" rpy="0.008 0.662 -1.725"/>
   </joint>
 <link name="realsense_holder1"/>
@@ -410,3 +410,4 @@
   <origin xyz="0 0 0" rpy="0 0 0"/>
 </xacro:sensor_d435>
+-->
 </robot>

Commit message: azure added

File: sharework_cembre_description/urdf/sharework_cembre_simplified.xacro (robot description, xacro)
@@ -35,4 +35,7 @@
 <xacro:property name="virtual_wall_width" value="0.001" />
 <xacro:property name="virtual_wall2_gap" value="1.10" />
+<xacro:property name="azure_size_x" value="0.150" />
+<xacro:property name="azure_size_y" value="0.300" />
+<xacro:property name="azure_size_z" value="0.400" />
 <!-- electric plug cabinet -->
 <xacro:property name="ec_size_x" value="0.40" />
@@ -401,4 +404,29 @@
 </link>
 <!-- CAMERA -->
+<joint name="upper_beam_to_azure" type="fixed">
+  <parent link="upper_beam"/>
+  <child link="azure"/>
+  <origin xyz="0 ${0.5*beam_size_y} 0"/>
+</joint>
+<link name="azure">
+ <visual>
+   <origin xyz="${0.5*azure_size_x} ${-0.5*azure_size_x} ${-0.5*azure_size_z}" rpy="0 0 0" />
+   <geometry>
+     <box size="${azure_size_x} ${azure_size_y} ${azure_size_z}" />
+   </geometry>
+   <material name="Grey">
+     <color rgba="${grey}"/>
+   </material>
+ </visual>
+ <collision>
+ <origin xyz="${0.5*azure_size_x} ${-0.5*azure_size_x} ${-0.5*azure_size_z}" rpy="0 0 0" />
+ <geometry>
+   <box size="${azure_size_x} ${azure_size_y} ${azure_size_z}" />
+ </geometry>
+ <material name="Grey">
+   <color rgba="${grey}"/>
+ </material>
+ </collision>
+</link>
 <!--<joint name="upper_beam_to_realsense2" type="fixed">
     <parent link="table"/>

Commit message: azure fixes

File: sharework_cembre_description/urdf/sharework_cembre_simplified.xacro (robot description, xacro)
@@ -411,5 +411,5 @@
 <link name="azure">
  <visual>
-   <origin xyz="${0.5*azure_size_x} ${-0.5*azure_size_x} ${-0.5*azure_size_z}" rpy="0 0 0" />
+   <origin xyz="${0.5*azure_size_x} ${-0.5*azure_size_y} ${-0.5*azure_size_z}" rpy="0 0 0" />
    <geometry>
      <box size="${azure_size_x} ${azure_size_y} ${azure_size_z}" />
@@ -420,5 +420,5 @@
  </visual>
  <collision>
- <origin xyz="${0.5*azure_size_x} ${-0.5*azure_size_x} ${-0.5*azure_size_z}" rpy="0 0 0" />
+ <origin xyz="${0.5*azure_size_x} ${-0.5*azure_size_y} ${-0.5*azure_size_z}" rpy="0 0 0" />
  <geometry>
    <box size="${azure_size_x} ${azure_size_y} ${azure_size_z}" />

Commit message: insert battery 3

File: sharework_cembre_description/urdf/sharework_cembre_simplified.xacro (robot description, xacro)
@@ -35,7 +35,10 @@
 <xacro:property name="virtual_wall_width" value="0.001" />
 <xacro:property name="virtual_wall2_gap" value="1.10" />
-<xacro:property name="azure_size_x" value="0.150" />
-<xacro:property name="azure_size_y" value="0.300" />
-<xacro:property name="azure_size_z" value="0.400" />
+<!-- <xacro:property name="azure_size_x" value="0.150" /> -->
+<!-- <xacro:property name="azure_size_y" value="0.300" /> -->
+<!-- <xacro:property name="azure_size_z" value="0.400" /> -->
+<xacro:property name="azure_size_x" value="0.300" />
+<xacro:property name="azure_size_y" value="0.330" />
+<xacro:property name="azure_size_z" value="0.440" />
 <!-- electric plug cabinet -->
 <xacro:property name="ec_size_x" value="0.40" />
@@ -45,4 +48,16 @@
 <xacro:property name="beech" value="0.952941176470588	0.694117647058823	0.392156862745098 1" />
 <xacro:property name="floor" value="0.4 0.4 0.5 1" />
+<link name="battery"/>
+<joint name="battery_joint" type="fixed">
+  <parent link="tool0"/>
+  <child link="battery"/>
+  <origin xyz="0 -0.047 0.205" rpy="1.5708 0 0"/>
+</joint>
+<link name="key"/>
+<joint name="key_joint" type="fixed">
+  <parent link="tool0"/>
+  <child link="key"/>
+  <origin xyz="0 0 0.235"/>
+</joint>
 <link name="world"/>
   <joint name="base_to_right_leg" type="fixed">
@@ -109,14 +124,14 @@
   </joint>
 <link name="lower_beam">
-   <visual>
+   <collision>
      <origin xyz="${0.5*beam_size_x} 0 ${-0.5*beam_size_z}" rpy="0 0 0" />
      <geometry>
-       <box size="${beam_size_x} ${beam_size_y} ${beam_size_z+2*anti_crushing_distance}" />
-     </geometry>
-     <material name="Grey">
-       <color rgba="${grey}"/>
-     </material>
-   </visual>
-   <collision>
+       <box size="${beam_size_x} ${beam_size_y} ${beam_size_z+2*anti_crushing_distance + 0.2}" />
+     </geometry>
+     <material name="Grey">
+       <color rgba="${grey}"/>
+     </material>
+   </collision>
+   <visual>
    <origin xyz="${0.5*beam_size_x} 0 ${-0.5*beam_size_z}" rpy="0 0 0" />
    <geometry>
@@ -126,5 +141,5 @@
      <color rgba="${grey}"/>
    </material>
-   </collision>
+ </visual>
 </link>
   <joint name="portal_to_upper_beam" type="fixed">
@@ -266,6 +281,6 @@
   shoulder_lift_lower_limit="${-pi}" shoulder_lift_upper_limit="0.052359878"
   elbow_joint_lower_limit="${-pi}" elbow_joint_upper_limit="${pi}"
-  wrist_1_lower_limit="${-pi}" wrist_1_upper_limit="${pi}"
-  wrist_2_lower_limit="${-pi}" wrist_2_upper_limit="${pi}"
+  wrist_1_lower_limit="${-2*pi}" wrist_1_upper_limit="${2*pi}"
+  wrist_2_lower_limit="${-2*pi}" wrist_2_upper_limit="${2*pi}"
   wrist_3_lower_limit="${-2*pi}" wrist_3_upper_limit="${2*pi}"
   transmission_hw_interface="$(arg transmission_hw_interface)"

Commit message: planner battery

File: sharework_cembre_description/urdf/sharework_cembre_simplified.xacro (robot description, xacro)
@@ -127,5 +127,5 @@
      <origin xyz="${0.5*beam_size_x} 0 ${-0.5*beam_size_z}" rpy="0 0 0" />
      <geometry>
-       <box size="${beam_size_x} ${beam_size_y} ${beam_size_z+2*anti_crushing_distance + 0.2}" />
+       <box size="${beam_size_x} ${beam_size_y} ${beam_size_z+2*anti_crushing_distance + 0.27}" />
      </geometry>
      <material name="Grey">

Commit message: ok

File: sharework_cembre_description/urdf/sharework_cembre_simplified.xacro (robot description, xacro)
@@ -60,4 +60,10 @@
   <origin xyz="0 0 0.235"/>
 </joint>
+<link name="ethernet"/>
+<joint name="ethernet_joint" type="fixed">
+  <parent link="tool0"/>
+  <child link="ethernet"/>
+  <origin xyz="0 0 0.226"/>
+</joint>
 <link name="world"/>
   <joint name="base_to_right_leg" type="fixed">
@@ -278,5 +284,5 @@
 <xacro:arg name="kinematics_config" default="$(find sharework_cembre_description)/config/cembre_ur10e.yaml"/>
 <xacro:ur10e_robot prefix="" joint_limited="true"
-  shoulder_pan_lower_limit="${-pi}" shoulder_pan_upper_limit="${pi}"
+  shoulder_pan_lower_limit="${-5.23599}" shoulder_pan_upper_limit="${5.23599}"
   shoulder_lift_lower_limit="${-pi}" shoulder_lift_upper_limit="0.052359878"
   elbow_joint_lower_limit="${-pi}" elbow_joint_upper_limit="${pi}"

Commit message: replanner controller

File: sharework_cembre_description/urdf/sharework_cembre_simplified.xacro (robot description, xacro)
@@ -7,2 +7,7 @@
   /> <!--DO NOT DELETE -->
 </robot>
+<!-- <xacro:macro name="robot_description" params=
+ "kinematics_config:=''$(find sharework_cembre_description)/config/cembre_ur10e.yaml'
+ transmission_hw_interface:=hardware_interface/PositionJointInterface "/>
+ kinematics_parameters_file="$(arg kinematics_config)"
+ transmission_hw_interface="$(arg transmission_hw_interface)" -->

Commit message: push from cari

File: sharework_cembre_description/urdf/sharework_cembre_simplified.xacro (robot description, xacro)
@@ -9,11 +9,11 @@
 <xacro:property name="table_size_x" value="0.600" />
 <xacro:property name="table_size_y" value="2.000" />
-<xacro:property name="table_size_z" value="0.040" />
+<xacro:property name="table_size_z" value="0.04" /> <!-- 0.04 -->>
 <xacro:property name="beam_size_x" value="${column_size_x}" />
 <xacro:property name="beam_size_y" value="${table_size_y}" />
-<xacro:property name="beam_size_z" value="${column_size_y}" />
+<xacro:property name="beam_size_z" value="${column_size_y+0.05}" /> <!-- added 0.05 -->>
 <xacro:property name="rail_size_x" value="0.36" />
 <xacro:property name="rail_size_y" value="3.224" />
-<xacro:property name="rail_size_z" value="0.17" />
+<xacro:property name="rail_size_z" value="0.14" />
 <xacro:property name="rail_distance" value="${0.162+0.5*rail_size_x}" />
 <xacro:property name="upper_beam_height" value="2.208" />
@@ -109,5 +109,5 @@
      <origin xyz="${0.5*beam_size_x} 0 ${-0.5*beam_size_z}" rpy="0 0 0" />
      <geometry>
-       <box size="${beam_size_x} ${beam_size_y} ${beam_size_z+2*anti_crushing_distance}" />
+       <box size="${beam_size_x} ${beam_size_y} ${beam_size_z}" />
      </geometry>
      <material name="Grey">
@@ -118,5 +118,5 @@
    <origin xyz="${0.5*beam_size_x} 0 ${-0.5*beam_size_z}" rpy="0 0 0" />
    <geometry>
-     <box size="${beam_size_x} ${beam_size_y} ${beam_size_z}" />
+     <box size="${beam_size_x} ${beam_size_y} ${beam_size_z+2*anti_crushing_distance}" />
    </geometry>
    <material name="Grey">
