Commit message: update rail size

File: sharework_cembre_description/urdf/sharework_cell.urdf.xacro (robot description, xacro)
@@ -25,6 +25,6 @@
 <xacro:property name="rail_size_x" value="0.36" />
 <xacro:property name="rail_size_y" value="3.224" />
-<xacro:property name="rail_size_z" value="0.17" />
-<xacro:property name="rail_distance" value="${0.162+0.5*rail_size_x}" />
+<xacro:property name="rail_size_z" value="0.14" />
+<xacro:property name="rail_distance" value="${0.12+0.5*rail_size_x}" />
 <xacro:property name="upper_beam_height" value="2.208" />
 <xacro:property name="guide_offset" value="${0.70-0.205}" />

Commit message: refine urdf

File: sharework_cembre_description/urdf/sharework_cell.urdf.xacro (robot description, xacro)
@@ -25,5 +25,5 @@
 <xacro:property name="rail_size_x" value="0.36" />
 <xacro:property name="rail_size_y" value="3.224" />
-<xacro:property name="rail_size_z" value="0.14" />
+<xacro:property name="rail_size_z" value="0.12" />
 <xacro:property name="rail_distance" value="${0.12+0.5*rail_size_x}" />
 <xacro:property name="upper_beam_height" value="2.208" />

Commit message: fix lower beam collision

File: sharework_cembre_description/urdf/sharework_cell.urdf.xacro (robot description, xacro)
@@ -117,14 +117,14 @@
 <link name="lower_beam">
    <visual>
-     <origin xyz="${0.5*beam_size_x} 0 ${-0.5*beam_size_z}" rpy="0 0 0" />
-     <geometry>
-       <box size="${beam_size_x} ${beam_size_y} ${beam_size_z+2*anti_crushing_distance}" />
-     </geometry>
-     <material name="Grey">
-       <color rgba="${grey}"/>
-     </material>
-   </visual>
-   <collision>
-   <origin xyz="${0.5*beam_size_x} 0 ${-0.5*beam_size_z}" rpy="0 0 0" />
+     <origin xyz="${0.5*beam_size_x} 0 ${-0.5*beam_size_z+0.012}" rpy="0 0 0" />
+     <geometry>
+       <box size="${beam_size_x} ${beam_size_y} ${beam_size_z}" />
+     </geometry>
+     <material name="Grey">
+       <color rgba="${grey}"/>
+     </material>
+   </visual>
+   <collision>
+   <origin xyz="${0.5*beam_size_x} 0 ${-0.5*beam_size_z+0.012}" rpy="0 0 0" />
    <geometry>
      <box size="${beam_size_x} ${beam_size_y} ${beam_size_z}" />

Commit message: changes from cembre

File: sharework_cembre_description/urdf/sharework_cell.urdf.xacro (robot description, xacro)
@@ -39,5 +39,5 @@
 <xacro:property name="wall_size_y" value="${2+table_size_y+2*column_size_y}" />
 <xacro:property name="wall_size_z" value="${column_size_z}" />
-<xacro:property name="wall_distance" value="0.500" />
+<xacro:property name="wall_distance" value="0.40" />
 <xacro:property name="floor_size_x" value="6" />
 <xacro:property name="floor_size_y" value="6" />
@@ -322,10 +322,10 @@
    </collision>
 </link>
-<joint name="wall_to_ec" type="fixed">
+<!-- <joint name="wall_to_ec" type="fixed">
     <parent link="wall"/>
-    <child link="ec"/>
+    <child link="electric_cabinet"/>
     <origin xyz="0 ${table_size_x*0.5} 0"/>
 </joint>
-<link name="ec">
+<link name="electric_cabinet">
    <visual>
      <origin xyz="${0.5*ec_size_x} ${0.5*ec_size_y} ${0.5*ec_size_z}" rpy="0 0 0" />
@@ -346,5 +346,5 @@
      </material>
    </collision>
-</link>
+</link> -->
 <joint name="portal_to_floor" type="fixed">
     <parent link="portal"/>
@@ -356,8 +356,8 @@
      <origin xyz="${0.5*floor_size_x-column_size_x-wall_distance} 0 ${-0.5*floor_size_z}" rpy="0 0 0" />
      <geometry>
-       <box size="${floor_size_x} ${floor_size_y} ${floor_size_z}" />
-     </geometry>
-     <material name="White">
-       <color rgba="1 1 1 1"/>
+       <box size="${floor_size_x} ${floor_size_y} ${floor_size_z+0.8}" />
+     </geometry>
+     <material name="White">
+       <color rgba="1 1 1 0.1"/>
      </material>
    </visual>

Commit message: fix

File: sharework_cembre_description/urdf/sharework_cell.urdf.xacro (robot description, xacro)
@@ -389,4 +389,30 @@
    </collision>
 </link>
+<!-- air manifold -->
+<joint name="table_to_air_manifold" type="fixed">
+    <parent link="table"/>
+    <child link="air_manifold"/>
+    <origin xyz="0.1 -0.05 0.35"/>
+  </joint>
+<link name="air_manifold">
+   <visual>
+     <origin xyz="0 0 0" rpy="0 0 0" />
+     <geometry>
+       <box size="0.2 0.2 0.4" />
+     </geometry>
+     <material name="White">
+       <color rgba="1 1 1 1"/>
+     </material>
+   </visual>
+   <collision>
+   <origin xyz="0 0 0" rpy="0 0 0" />
+   <geometry>
+     <box size="0.2 0.2 0.4" />
+   </geometry>
+   <material name="White">
+     <color rgba="1 1 1 1"/>
+   </material>
+   </collision>
+</link>
 <!-- Virtual Wall -->
 <joint name="virtual_wall_1_joint" type="fixed">
@@ -422,4 +448,54 @@
   </collision>
 </link>
+<joint name="thing_on_wall_joint" type="fixed">
+    <parent link="world"/>
+    <child link="thing_on_wall"/>
+    <origin xyz="0 0 0.0"/>
+  </joint>
+<link name="thing_on_wall">
+  <visual>
+    <origin xyz="-0.2 -0.95 1.35" rpy="0 0 0" />
+    <geometry>
+      <box size="0.5 0.1 0.3" />
+    </geometry>
+     <material name="Grey">
+       <color rgba="${grey}"/>
+     </material>
+  </visual>
+  <collision>
+    <origin xyz="-0.2 -0.95 1.35" rpy="0 0 0" />
+    <geometry>
+      <box size="0.5 0.1 0.3" />
+    </geometry>
+     <material name="Grey">
+       <color rgba="${grey}"/>
+     </material>
+  </collision>
+</link>
+<joint name="computer_screen_joint" type="fixed">
+    <parent link="world"/>
+    <child link="computer_screen"/>
+    <origin xyz="0 0 0.0"/>
+  </joint>
+<link name="computer_screen">
+  <visual>
+    <origin xyz="0.15 1.2 1.5" rpy="0 0 0" />
+    <geometry>
+      <box size="0.2 0.5 0.5" />
+    </geometry>
+     <material name="Grey">
+       <color rgba="${grey}"/>
+     </material>
+  </visual>
+  <collision>
+    <origin xyz="0.15 1.2 1.5" rpy="0 0 0" />
+    <geometry>
+      <box size="0.2 0.5 0.5" />
+    </geometry>
+     <material name="Grey">
+       <color rgba="${grey}"/>
+     </material>
+  </collision>
+</link>
 </xacro:macro>
 </robot>

Commit message: completed description package

File: sharework_cembre_description/urdf/sharework_cell.urdf.xacro (robot description, xacro)
@@ -1,17 +1,16 @@
 <?xml version="1.0"?>
-<robot xmlns:xacro="http://ros.org/wiki/xacro" name="sharework_cell" >
-<xacro:macro name="sharework_cell" params=
- "simplified
-  prefix:=''
-  joint_limits_parameters_file:='$(find sharework_cembre_description)/config/joint_limits.yaml'
-  kinematics_parameters_file:='$(find sharework_cembre_description)/config/cembre_ur10e.yaml'
-  physical_parameters_file:='$(find ur_description)/config/ur10e/physical_parameters.yaml'
-  visual_parameters_file:='$(find ur_description)/config/ur10e/visual_parameters.yaml'
-  transmission_hw_interface:=hardware_interface/PositionJointInterface
-  safety_limits:=false
-  safety_pos_margin:=0.15
-  safety_k_position:=20 ">
-<xacro:include filename="$(find realsense2_description)/urdf/_d435.urdf.xacro" />
-<!-- <xacro:include filename="$(find robotiq_2f_85_gripper_visualization)/urdf/robotiq_arg2f_85_model_macro.xacro" /> -->
+<robot xmlns:xacro="http://ros.org/wiki/xacro" name="sharework_cell_macro" >
+<xacro:macro
+  name="sharework_cell"
+  params=
+    "joint_limits_parameters_file:='$(find sharework_cembre_description)/config/joint_limits.yaml'
+     kinematics_parameters_file:='$(find sharework_cembre_description)/config/cembre_ur10e.yaml'
+     safety_limits:=false
+     safety_pos_margin:=0.15
+     safety_k_position:=20
+     zed_camera_name:='zed'
+     zed_camera_model:='zed2'
+    "
+>
 <xacro:property name="column_size_x" value="0.580" />
 <xacro:property name="column_size_y" value="0.120" />
@@ -52,5 +51,4 @@
 <xacro:property name="grey" value="0.517647058823529	0.529411764705882	0.537254901960784 1" />
 <xacro:property name="beech" value="0.952941176470588	0.694117647058823	0.392156862745098 1" />
-<xacro:property name="floor" value="0.4 0.4 0.5 1" />
 <link name="world"/>
 <joint name="base_to_right_leg" type="fixed">
@@ -265,36 +263,4 @@
    </collision>
 </link>
-<!-- ur10e -->
-<xacro:if value="${simplified == True}">
-  <xacro:include filename="$(find ur10e_robotiq_simplified_description)/urdf/ur10e_robotiq.urdf.xacro"/>
-  <xacro:ur10e_robotiq_simplified
-    prefix = "${prefix}"
-    joint_limits_parameters_file="${joint_limits_parameters_file}"
-    kinematics_parameters_file="${kinematics_parameters_file}"
-    physical_parameters_file="${physical_parameters_file}"
-    transmission_hw_interface="${transmission_hw_interface}"
-    safety_limits="${safety_limits}"
-    safety_pos_margin="${safety_pos_margin}"
-    safety_k_position="${safety_k_position}"
-  />
-</xacro:if>
-<xacro:if value="${simplified == False}">
-  <xacro:include filename="$(find ur10e_robotiq_description)/urdf/ur10e_robotiq.urdf.xacro"/>
-  <xacro:ur10e_robotiq
-    prefix = "${prefix}"
-    joint_limits_parameters_file="${joint_limits_parameters_file}"
-    kinematics_parameters_file="${kinematics_parameters_file}"
-    physical_parameters_file="${physical_parameters_file}"
-    transmission_hw_interface="${transmission_hw_interface}"
-    safety_limits="${safety_limits}"
-    safety_pos_margin="${safety_pos_margin}"
-    safety_k_position="${safety_k_position}"
-  />
-</xacro:if>
-<joint name="cursor_to_base" type="fixed">
-  <parent link="cursor" />
-  <child link = "base_link" />
-  <origin xyz="0.0 0.0 0.0" rpy="${pi} 0.0 ${0.5*pi}" />
-</joint>
 <!-- walls  -->
 <joint name="portal_to_wall" type="fixed">
@@ -323,5 +289,5 @@
    </collision>
 </link>
-<!-- <joint name="wall_to_ec" type="fixed">
+<joint name="wall_to_ec" type="fixed">
     <parent link="wall"/>
     <child link="electric_cabinet"/>
@@ -347,5 +313,5 @@
      </material>
    </collision>
-</link> -->
+</link>
 <joint name="portal_to_floor" type="fixed">
     <parent link="portal"/>
@@ -365,5 +331,5 @@
 </link>
 <!-- Screw driver -->
-<joint name="table_to_screwdriver_holder" type="fixed">
+<!-- <joint name="table_to_screwdriver_holder" type="fixed">
     <parent link="table"/>
     <child link="screwdriver_holder"/>
@@ -389,7 +355,7 @@
    </material>
    </collision>
-</link>
+</link> -->
 <!-- air manifold -->
-<joint name="table_to_air_manifold" type="fixed">
+<!-- <joint name="table_to_air_manifold" type="fixed">
     <parent link="table"/>
     <child link="air_manifold"/>
@@ -415,5 +381,5 @@
    </material>
    </collision>
-</link>
+</link> -->
 <!-- Virtual Wall -->
 <joint name="virtual_wall_1_joint" type="fixed">
@@ -475,8 +441,8 @@
 </link>
 <joint name="computer_screen_joint" type="fixed">
-    <parent link="world"/>
-    <child link="computer_screen"/>
-    <origin xyz="0 0 0.0"/>
-  </joint>
+  <parent link="world"/>
+  <child link="computer_screen"/>
+  <origin xyz="0 0 0.0"/>
+</joint>
 <link name="computer_screen">
   <visual>
@@ -499,4 +465,71 @@
   </collision>
 </link>
+<!-- ur10e -->
+<xacro:include filename="$(find ur10e_robotiq_description)/urdf/ur10e_robotiq.urdf.xacro"/>
+<xacro:ur10e_robotiq
+  parent='cursor'
+  joint_limits_parameters_file="${joint_limits_parameters_file}"
+  kinematics_parameters_file="${kinematics_parameters_file}"
+  safety_limits="${safety_limits}"
+  safety_pos_margin="${safety_pos_margin}"
+  safety_k_position="${safety_k_position}"
+  origin_xyz="0.0 0.0 0.0"
+  origin_rpy="${pi} 0.0 ${0.5*pi}"
+  initial_positions="${dict(shoulder_pan_joint=1.570796327,
+                            shoulder_lift_joint=-2.443460953,
+                            elbow_joint=2.443460953,
+                            wrist_1_joint=-1.570796327,
+                            wrist_2_joint=1.570796327,
+                            wrist_3_joint=0.0,
+                            finger_joint=-0.04)}"
+/>
+<!-- ZED camera -->
+<joint name="zed_world_joint" type="floating">
+  <parent link="world"/>
+  <child link="${zed_camera_name}_camera_link"/>
+  <origin xyz="0.0 0.0 0.0"
+          rpy="0.0 0.0 0.0" />
+</joint>
+<xacro:include filename="$(find zed_wrapper)/urdf/zed_macro.urdf.xacro" />
+<xacro:arg name="custom_baseline"  default="0.0" />
+<!-- If GNSS fusion is enabled the position of the antenna with respect to the camera mount point is required -->
+<xacro:arg name="enable_gnss"   default="false" />
+<xacro:arg name="gnss_x" default="0.0" />
+<xacro:arg name="gnss_y" default="0.0" />
+<xacro:arg name="gnss_z" default="0.0" />
+<xacro:zed_camera name="${zed_camera_name}" model="${zed_camera_model}" custom_baseline="$(arg custom_baseline)" enable_gnss="$(arg enable_gnss)">
+	    <origin xyz="$(arg gnss_x) $(arg gnss_y) $(arg gnss_z)" rpy="0 0 0"/>
+</xacro:zed_camera>
+<!-- Realsense cameras -->
+<link name="rs1_camera_link" />
+<joint name="rs1_world_joint" type="floating">
+  <parent link="world"/>
+  <child link="rs1_camera_link"/>
+  <origin xyz="0.0 0.0 0.0"
+          rpy="0.0 0.0 0.0" />
+</joint>
+<xacro:include filename="$(find realsense2_description)/urdf/_d435.urdf.xacro" />
+<xacro:sensor_d435
+    parent='rs1_camera_link'
+    name="rs1"
+  >
+  <origin xyz="0.0 0.0 0.0"
+          rpy="0.0 0.0 0.0" />
+</xacro:sensor_d435>
+<link name="rs2_camera_link" />
+<joint name="rs2_world_joint" type="floating">
+  <parent link="world"/>
+  <child link="rs2_camera_link"/>
+  <origin xyz="0.0 0.0 0.0"
+          rpy="0.0 0.0 0.0" />
+</joint>
+<xacro:include filename="$(find realsense2_description)/urdf/_d435i.urdf.xacro" />
+<xacro:sensor_d435
+    parent='rs2_camera_link'
+    name="rs2"
+  >
+  <origin xyz="0.0 0.0 0.0"
+          rpy="0.0 0.0 0.0" />
+</xacro:sensor_d435>
 </xacro:macro>
 </robot>
