Commit message: jazzy clean

File: sharework_cembre_description/urdf/sharework_cell.urdf.xacro (robot description, xacro)
@@ -7,5 +7,4 @@
   <xacro:arg name="zed_camera_name"              default="zed"/>
   <xacro:arg name="zed_camera_model"             default="zed2"/>
-  <xacro:arg name="robot_parent_link"            default="cursor"/>
   <xacro:arg name="robot_origin_x"               default="0.0"/>
   <xacro:arg name="robot_origin_y"               default="0.0"/>
@@ -31,9 +30,9 @@
   <xacro:arg name="robotiq_activate_gripper_by_default" default="1" /> <!-- 0: false, 1: true -->
   <!-- UR properties -->
-  <xacro:property name="joint_limit_params"        value="$(find ur_robotiq_description)/config/$(arg ur_type)/joint_limits.yaml"/>
-  <xacro:property name="kinematics_params"         value="$(find ur_robotiq_description)/config/$(arg ur_type)/default_kinematics.yaml"/>
-  <xacro:property name="physical_params"           value="$(find ur_robotiq_description)/config/$(arg ur_type)/physical_parameters.yaml"/>
-  <xacro:property name="visual_params"             value="$(find ur_robotiq_description)/config/$(arg ur_type)/visual_parameters.yaml"/>
-  <xacro:property name="initial_positions_file"    value="$(find ur_robotiq_description)/config/ur10e/initial_positions.yaml"/>
+  <xacro:property name="joint_limit_params"        value="$(find sharework_cembre_description)/config/joint_limits.yaml"/>
+  <xacro:property name="kinematics_params"         value="$(find sharework_cembre_description)/config/default_kinematics.yaml"/>
+  <xacro:property name="physical_params"           value="$(find sharework_cembre_description)/config/physical_parameters.yaml"/>
+  <xacro:property name="visual_params"             value="$(find sharework_cembre_description)/config/visual_parameters.yaml"/>
+  <xacro:property name="initial_positions_file"    value="$(find sharework_cembre_description)/config/initial_positions.yaml"/>
   <xacro:property name="transmission_hw_interface" value=""/>
   <xacro:property name="safety_limits"             value="false"/>
@@ -75,5 +74,4 @@
     fake_robot="$(arg fake_robot)"
     fake_gripper="$(arg fake_gripper)"
-    robot_parent_link="$(arg robot_parent_link)"
     robot_origin_x="$(arg robot_origin_x)"
     robot_origin_y="$(arg robot_origin_y)"
@@ -118,5 +116,5 @@
     trajectory_port="${trajectory_port}"
     non_blocking_read="${non_blocking_read}"
-    keep_alive_count="${keep_alive_count}"
+    robot_receive_timeout="${robot_receive_timeout}"
     robotiq_sim_isaac="${robotiq_sim_isaac}"
     robotiq_isaac_joint_commands="${robotiq_isaac_joint_commands}"

File: sharework_cembre_description/urdf/sharework_cell.xacro (robot description, xacro)
@@ -7,5 +7,4 @@
   fake_robot:=true
   fake_gripper:=true
-  robot_parent_link:='cursor'
   robot_origin_x:='0.0'
   robot_origin_y:='0.0'
@@ -13,6 +12,6 @@
   robot_origin_roll:='${pi}'
   robot_origin_pitch:='0.0'
-  robot_origin_yaw:='0.0'
-  ur_type:='ur10e'
+  robot_origin_yaw:='${pi/2}'
+  ur_type:='$(arg ur_type)'
   robot_name:='$(arg ur_type)'
   robot_tf_prefix:='$(arg ur_type)'
@@ -31,10 +30,10 @@
   headless_mode:=false
   initial_positions:=${dict(
-                        shoulder_pan_joint=0.0,
-                        shoulder_lift_joint=-1.57,
-                        elbow_joint=0.0,
-                        wrist_1_joint=-1.57,
-                        wrist_2_joint=0.0,
-                        wrist_3_joint=0.0,
+                        ur10e_shoulder_pan_joint=0.0,
+                        ur10e_shoulder_lift_joint=-1.57,
+                        ur10e_elbow_joint=0.0,
+                        ur10e_wrist_1_joint=-1.57,
+                        ur10e_wrist_2_joint=0.0,
+                        ur10e_wrist_3_joint=0.0,
                         left_knuckle_joint=0.0
                       )}
@@ -58,5 +57,5 @@
   trajectory_port:=50003
   non_blocking_read:=true
-  keep_alive_count:=2
+  robot_receive_timeout:=0.04
   robotiq_sim_isaac:=false
   robotiq_isaac_joint_commands:=/isaac_joint_commands
@@ -69,116 +68,67 @@
   robotiq_connection_timeout:=30000
   robotiq_activate_gripper_by_default:=1">
-<!-- ZED camera args-->
-<xacro:property name="custom_baseline"  value="0.0" />
-<!-- If GNSS fusion is enabled the position of the antenna with respect to the camera mount point is required -->
-<xacro:property name="enable_gnss"      value="false" />
-<xacro:property name="gnss_x"           value="0.0" />
-<xacro:property name="gnss_y"           value="0.0" />
-<xacro:property name="gnss_z"           value="0.0" />
-<!-- Geometric properties -->
-<xacro:property name="column_size_x" value="0.580" />
-<xacro:property name="column_size_y" value="0.120" />
-<xacro:property name="column_size_z" value="3.000" />
-<xacro:property name="table_height" value="0.895" />
-<xacro:property name="table_size_x" value="0.600" />
-<xacro:property name="table_size_y" value="2.000" />
-<xacro:property name="table_size_z" value="0.040" />
-<xacro:property name="beam_size_x" value="${column_size_x}" />
-<xacro:property name="beam_size_y" value="${table_size_y}" />
-<xacro:property name="beam_size_z" value="${column_size_y}" />
-<xacro:property name="rail_size_x" value="0.36" />
-<xacro:property name="rail_size_y" value="3.224" />
-<xacro:property name="rail_size_z" value="0.12" />
-<xacro:property name="rail_distance" value="${0.12+0.5*rail_size_x}" />
-<xacro:property name="upper_beam_height" value="2.208" />
-<xacro:property name="guide_offset" value="${0.70-0.205}" />
-<xacro:property name="cursor_size" value="0.280" />
-<xacro:property name="guide_size_x" value="${cursor_size}" />
-<xacro:property name="guide_size_y" value="${beam_size_y}" />
-<xacro:property name="guide_size_z" value="0.14" />
-<xacro:property name="guide_distance_x" value="0.185" />
-<xacro:property name="anti_crushing_distance" value="0.040" />
-<xacro:property name="guide_distance_y" value="${0.385+0.041}" />
-<xacro:property name="wall_size_x" value="0.1" />
-<xacro:property name="wall_size_y" value="${2+table_size_y+2*column_size_y}" />
-<xacro:property name="wall_size_z" value="${column_size_z}" />
-<xacro:property name="wall_distance" value="0.40" />
-<xacro:property name="floor_size_x" value="6" />
-<xacro:property name="floor_size_y" value="6" />
-<xacro:property name="floor_size_z" value="0.01" />
-<xacro:property name="virtual_wall_width" value="0.001" />
-<xacro:property name="virtual_wall2_gap" value="1.10" />
-<!-- electric plug cabinet -->
-<xacro:property name="ec_size_x" value="0.40" />
-<xacro:property name="ec_size_y" value="0.70" />
-<xacro:property name="ec_size_z" value="2.00" />
-<xacro:property name="grey" value="0.517647058823529	0.529411764705882	0.537254901960784 1" />
-<xacro:property name="beech" value="0.952941176470588	0.694117647058823	0.392156862745098 1" />
   <xacro:include filename="$(find sharework_cembre_description)/urdf/sharework_fixed_parts.xacro" />
   <xacro:sharework_fixed_parts />
   <xacro:include filename="$(find sharework_cembre_description)/urdf/sharework_sensors.xacro"/>
   <xacro:sharework_sensors
-          fake_cameras="${fake_cameras}"
+    zed_camera_name="${zed_camera_name}"
+    zed_camera_model="${zed_camera_model}"
+    fake_cameras="${fake_cameras}"
   />
-  <!-- ur10e + robotiq gripper -->
-<xacro:include filename="$(find ur_robotiq_description)/urdf/ur_robotiq.xacro"/>
-<xacro:ur_robotiq
-        fake_ur="${fake_robot}"
-  fake_gripper="${fake_gripper}"
-  parent_link="${robot_parent_link}"
-  origin_x="${robot_origin_x}"
-  origin_y="${robot_origin_y}"
-  origin_z="${robot_origin_z}"
-  origin_roll="${robot_origin_roll}"
-  origin_pitch="${robot_origin_pitch}"
-  origin_yaw="${robot_origin_yaw}"
-  ur_type="${ur_type}"
-  robot_name="${robot_name}"
-  tf_prefix="${robot_tf_prefix}"
-  joint_limits_parameters_file="${joint_limit_params}"
-  kinematics_parameters_file="${kinematics_params}"
-  physical_parameters_file="${physical_params}"
-  visual_parameters_file="${visual_params}"
-  safety_limits="${safety_limits}"
-  safety_pos_margin="${safety_pos_margin}"
-  safety_k_position="${safety_k_position}"
-  generate_ros2_control_tag="${generate_ros2_control_tag}"
-  transmission_hw_interface="${transmission_hw_interface}"
-  fake_sensor_commands="${fake_sensor_commands}"
-  sim_gazebo="${sim_gazebo}"
-  sim_ignition="${sim_ignition}"
-  headless_mode="${headless_mode}"
-  initial_positions="${initial_positions}"
-  use_tool_communication="${use_tool_communication}"
-  tool_voltage="${tool_voltage}"
-  tool_parity="${tool_parity}"
-  tool_baud_rate="${tool_baud_rate}"
-  tool_stop_bits="${tool_stop_bits}"
-  tool_rx_idle_chars="${tool_rx_idle_chars}"
-  tool_tx_idle_chars="${tool_tx_idle_chars}"
-  tool_device_name="${tool_device_name}"
-  tool_tcp_port="${tool_tcp_port}"
-  robot_ip="${robot_ip}"
-  script_filename="${script_filename}"
-  output_recipe_filename="${output_recipe_filename}"
-  input_recipe_filename="${input_recipe_filename}"
-  reverse_port="${reverse_port}"
-  script_sender_port="${script_sender_port}"
-  reverse_ip="${reverse_ip}"
-  script_command_port="${script_command_port}"
-  trajectory_port="${trajectory_port}"
-  non_blocking_read="${non_blocking_read}"
-  keep_alive_count="${keep_alive_count}"
-  robotiq_sim_ignition="${sim_ignition}"
-  robotiq_sim_isaac="${robotiq_sim_isaac}"
-  robotiq_isaac_joint_commands="${robotiq_isaac_joint_commands}"
-  robotiq_isaac_joint_states="${robotiq_isaac_joint_states}"
-  robotiq_mock_sensor_commands="${robotiq_mock_sensor_commands}"
-  robotiq_include_ros2_control="${robotiq_include_ros2_control}"
-  robotiq_use_socket_communication="${robotiq_use_socket_communication}"
-  robotiq_ip_address="${robotiq_ip_address}"
-  robotiq_port="${robotiq_port}"
-  robotiq_connection_timeout="${robotiq_connection_timeout}"
-  robotiq_activate_gripper_by_default="${robotiq_activate_gripper_by_default}"/>
+  <xacro:include filename="$(find sharework_cembre_description)/urdf/moving_parts.xacro"/>
+  <xacro:sharework_moving_parts
+    parent="cursor"
+    fake_gripper="${fake_gripper}"
+    ur_type="${ur_type}"
+    robot_name="${robot_name}"
+    robot_tf_prefix="${robot_tf_prefix}"
+    joint_limits_parameters_file="${joint_limits_parameters_file}"
+    kinematics_parameters_file="${kinematics_parameters_file}"
+    physical_parameters_file="${physical_parameters_file}"
+    visual_parameters_file="${visual_parameters_file}"
+    safety_limits="${safety_limits}"
+    safety_pos_margin="${safety_pos_margin}"
+    safety_k_position="${safety_k_position}"
+    generate_ros2_control_tag="${generate_ros2_control_tag}"
+    transmission_hw_interface="${transmission_hw_interface}"
+    use_mock_hardware="${fake_robot}"
+    mock_sensor_commands="${fake_robot or fake_sensor_commands}"
+    initial_positions="${initial_positions}"
+    headless_mode="${headless_mode}"
+    robot_ip="${robot_ip}"
+    script_filename="${script_filename}"
+    output_recipe_filename="${output_recipe_filename}"
+    input_recipe_filename="${input_recipe_filename}"
+    reverse_ip="${reverse_ip}"
+    script_command_port="${script_command_port}"
+    reverse_port="${reverse_port}"
+    script_sender_port="${script_sender_port}"
+    trajectory_port="${trajectory_port}"
+    non_blocking_read="${non_blocking_read}"
+    robot_receive_timeout="${robot_receive_timeout}"
+    use_tool_communication="${use_tool_communication}"
+    tool_voltage="${tool_voltage}"
+    tool_parity="${tool_parity}"
+    tool_baud_rate="${tool_baud_rate}"
+    tool_stop_bits="${tool_stop_bits}"
+    tool_rx_idle_chars="${tool_rx_idle_chars}"
+    tool_tx_idle_chars="${tool_tx_idle_chars}"
+    tool_device_name="${tool_device_name}"
+    tool_tcp_port="${tool_tcp_port}"
+    robotiq_sim_ignition="${sim_ignition}"
+    robotiq_sim_isaac="${robotiq_sim_isaac}"
+    robotiq_isaac_joint_commands="${robotiq_isaac_joint_commands}"
+    robotiq_isaac_joint_states="${robotiq_isaac_joint_states}"
+    robotiq_mock_sensor_commands="${robotiq_mock_sensor_commands}"
+    robotiq_include_ros2_control="${robotiq_include_ros2_control}"
+    robotiq_use_socket_communication="${robotiq_use_socket_communication}"
+    robotiq_ip_address="${robotiq_ip_address}"
+    robotiq_port="${robotiq_port}"
+    robotiq_connection_timeout="${robotiq_connection_timeout}"
+    robotiq_activate_gripper_by_default="${robotiq_activate_gripper_by_default}"
+    >
+    <origin xyz="${robot_origin_x} ${robot_origin_y} ${robot_origin_z}"
+            rpy="${robot_origin_roll} ${robot_origin_pitch} ${robot_origin_yaw}" />
+  </xacro:sharework_moving_parts>
 </xacro:macro>
 </robot>

File: sharework_cembre_description/urdf/sharework_sensors.xacro (robot description, xacro)
@@ -1,131 +1,53 @@
 <?xml version="1.0"?>
-<robot xmlns:xacro="http://ros.org/wiki/xacro" name="sharework_fixed_parts">
-    <xacro:macro name="sharework_sensors" params="
+<robot xmlns:xacro="http://ros.org/wiki/xacro" name="sharework_sensors">
+  <xacro:include filename="$(find sharework_cembre_description)/urdf/zed_camera.xacro" />
+  <xacro:include filename="$(find sharework_cembre_description)/urdf/realsense_camera.xacro" />
+  <!-- ##################################################################
+       Orchestratore dei sensori della cella. Ogni telecamera fisica
+       e' una singola chiamata a macro: aggiungere/rimuovere una camera
+       significa aggiungere/rimuovere una call qui sotto, senza toccare
+       la logica fake/reale (che vive in zed_camera.xacro / realsense_camera.xacro)
+       ################################################################## -->
+  <xacro:macro name="sharework_sensors" params="
     zed_camera_name:='zed'
     zed_camera_model:='zed2'
     fake_cameras:=true
   ">
-        <!-- ZED camera args -->
-        <xacro:property name="custom_baseline"  value="0.0" />
-        <xacro:property name="enable_gnss"      value="false" />
-        <xacro:property name="gnss_x"           value="0.0" />
-        <xacro:property name="gnss_y"           value="0.0" />
-        <xacro:property name="gnss_z"           value="0.0" />
-        <!-- #############################################
-             ZED mount to world
-             NOTE: camera_link is created either by the real zed macro
-                   (fake_cameras=false) OR by our fake block (true)
-             ############################################# -->
-        <joint name="zed_world_joint" type="fixed">
-            <parent link="world"/>
-            <child link="${zed_camera_name}_camera_link"/>
-            <!-- Replace with calibration -->
-            <origin xyz="0.0937849 -0.929844 2.30862"
-                    rpy="0.8165 0.9372 0.7201" />
-        </joint>
-        <!-- Real ZED -->
-        <xacro:if value="${not fake_cameras}">
-            <xacro:include filename="$(find zed_wrapper)/urdf/zed_macro.urdf.xacro" />
-            <xacro:zed_camera
-                    name="${zed_camera_name}"
-                    model="${zed_camera_model}"
-                    custom_baseline="${custom_baseline}"
-                    enable_gnss="${enable_gnss}">
-                <!-- GNSS antenna pose wrt camera mount point (if used) -->
-                <origin xyz="${gnss_x} ${gnss_y} ${gnss_z}"
-                        rpy="0 0 0"/>
-            </xacro:zed_camera>
-        </xacro:if>
-        <!-- Fake ZED frames -->
-        <xacro:if value="${fake_cameras}">
-            <!-- Minimal link tree so TF consumers can resolve optical frame -->
-            <link name="${zed_camera_name}_camera_link"/>
-            <link name="${zed_camera_name}_camera_optical_frame"/>
-            <joint name="${zed_camera_name}_camera_optical_joint" type="fixed">
-                <parent link="${zed_camera_name}_camera_link"/>
-                <child link="${zed_camera_name}_camera_optical_frame"/>
-                <!-- Typical optical frame rotation (REP-103 / REP-105 style) -->
-                <origin xyz="0 0 0" rpy="-1.57079632679 0 -1.57079632679"/>
-            </joint>
-            zed_camera_center
-            <link name="${zed_camera_name}_camera_center" />
-            <joint name="${zed_camera_name}_camera_center_joint" type="fixed">
-                <parent link="${zed_camera_name}_camera_link"/>
-                <child link="${zed_camera_name}_camera_center"/>
-                <!-- Replace with calibration -->
-                <origin xyz="0.0 0.0 0.0"
-                        rpy="0.0 0.0 0.0" />
-            </joint>
-        </xacro:if>
-        <!-- #############################################
-             Realsense 1
-             ############################################# -->
-        <link name="rs1_camera_link" />
-        <joint name="rs1_world_joint" type="fixed">
-            <parent link="world"/>
-            <child link="rs1_camera_link"/>
-            <!-- Replace with calibration -->
-            <origin xyz="0.845205 1.15052 2.57347"
-                    rpy="0.0773 0.773 -1.553" />
-        </joint>
-        <!-- Real RS1 -->
-        <xacro:if value="${not fake_cameras}">
-            <xacro:include filename="$(find realsense2_description)/urdf/_d435.urdf.xacro" />
-            <xacro:sensor_d435 parent="rs1_camera_link" name="rs1">
-                <origin xyz="0 0 0" rpy="0 0 0" />
-            </xacro:sensor_d435>
-        </xacro:if>
-        <!-- Fake RS1 optical frame -->
-        <xacro:if value="${fake_cameras}">
-            <link name="rs1_camera_optical_frame"/>
-            <joint name="rs1_camera_optical_joint" type="fixed">
-                <parent link="rs1_camera_link"/>
-                <child link="rs1_camera_optical_frame"/>
-                <origin xyz="0 0 0" rpy="-1.57079632679 0 -1.57079632679"/>
-            </joint>
-            <link name="rs1_link" />
-            <joint name="rs1_camera_joint" type="fixed">
-                <parent link="rs1_camera_link"/>
-                <child link="rs1_link"/>
-                <!-- Replace with calibration -->
-                <origin xyz="0.0 0.0 0.0"
-                        rpy="0.0 0.0 0.0" />
-            </joint>
-        </xacro:if>
-        <!-- #############################################
-             Realsense 2
-             ############################################# -->
-        <link name="rs2_camera_link" />
-        <joint name="rs2_world_joint" type="fixed">
-            <parent link="world"/>
-            <child link="rs2_camera_link"/>
-            <!-- Replace with calibration -->
-            <origin xyz="0.649999 -1.16584 2.63428"
-                    rpy="-0.0696 0.795 1.502" />
-        </joint>
-        <!-- Real RS2 -->
-        <xacro:if value="${not fake_cameras}">
-            <xacro:include filename="$(find realsense2_description)/urdf/_d435i.urdf.xacro" />
-            <xacro:sensor_d435 parent="rs2_camera_link" name="rs2">
-                <origin xyz="0 0 0" rpy="0 0 0" />
-            </xacro:sensor_d435>
-        </xacro:if>
-        <!-- Fake RS2 optical frame -->
-        <xacro:if value="${fake_cameras}">
-            <link name="rs2_camera_optical_frame"/>
-            <joint name="rs2_camera_optical_joint" type="fixed">
-                <parent link="rs2_camera_link"/>
-                <child link="rs2_camera_optical_frame"/>
-                <origin xyz="0 0 0" rpy="-1.57079632679 0 -1.57079632679"/>
-            </joint>
-            <link name="rs2_link" />
-            <joint name="rs2_camera_joint" type="fixed">
-                <parent link="rs2_camera_link"/>
-                <child link="rs2_link"/>
-                <!-- Replace with calibration -->
-                <origin xyz="0.0 0.0 0.0"
-                        rpy="0.0 0.0 0.0" />
-            </joint>
-        </xacro:if>
-    </xacro:macro>
+    <!-- ============================== ZED ============================== -->
+    <xacro:sharework_zed_camera
+            camera_name="${zed_camera_name}"
+            camera_model="${zed_camera_model}"
+            fake="${fake_cameras}"
+            parent="world"
+            origin_xyz="0.0937849 -0.929844 2.30862"
+            origin_rpy="0.8165 0.9372 0.7201"
+    />
+    <!-- ========================= RealSense 1 ============================ -->
+    <xacro:sharework_realsense_camera
+            name="rs1"
+            fake="${fake_cameras}"
+            parent="world"
+            origin_xyz="0.845205 1.15052 2.57347"
+            origin_rpy="0.0773 0.773 -1.553"
+            realsense_model="d435"
+    />
+    <!-- ========================= RealSense 2 ============================ -->
+    <xacro:sharework_realsense_camera
+            name="rs2"
+            fake="${fake_cameras}"
+            parent="world"
+            origin_xyz="0.649999 -1.16584 2.63428"
+            origin_rpy="-0.0696 0.795 1.502"
+            realsense_model="d435i"
+    />
+    <!-- Per aggiungere una terza RealSense basta una call in piu', es.:
+    <xacro:sharework_realsense_camera
+            name="rs3"
+            fake="${fake_cameras}"
+            parent="world"
+            origin_xyz="x y z"
+            origin_rpy="r p y"
+    />
+    -->
+  </xacro:macro>
 </robot>
