Commit message: pos to vel ctrl

File: sharework_cembre_description/urdf/old/sharework_cembre.xacro (robot description, xacro)
@@ -107,14 +107,14 @@
 <link name="lower_beam">
    <visual>
-     <origin xyz="${0.5*beam_size_x} 0 ${-0.5*beam_size_z}" rpy="0 0 0" />
-     <geometry>
-       <box size="${beam_size_x} ${beam_size_y} ${beam_size_z+2*anti_crushing_distance}" />
-     </geometry>
-     <material name="Grey">
-       <color rgba="${grey}"/>
-     </material>
-   </visual>
-   <collision>
-   <origin xyz="${0.5*beam_size_x} 0 ${-0.5*beam_size_z}" rpy="0 0 0" />
+     <origin xyz="${0.5*beam_size_x} 0 ${-0.5*beam_size_z+0.015}" rpy="0 0 0" />
+     <geometry>
+       <box size="${beam_size_x} ${beam_size_y} ${beam_size_z}" />
+     </geometry>
+     <material name="Grey">
+       <color rgba="${grey}"/>
+     </material>
+   </visual>
+   <collision>
+   <origin xyz="${0.5*beam_size_x} 0 ${-0.5*beam_size_z+0.015}" rpy="0 0 0" />
    <geometry>
      <box size="${beam_size_x} ${beam_size_y} ${beam_size_z}" />
